Commit message: Update robot_core.xacro

File: Kobuki_sim/description/robot_core.xacro (robot description, xacro)
@@ -46,5 +46,5 @@
           <!-- new mesh -->
           <!--mesh filename="file://$(find articubot_one)/meshes/microwave.stl" scale="0.01 0.01 0.01"/-->
-          <mesh filename="file://$(find articubot_one)/meshes/kobuki_base.stl" scale="0.01 0.01 0.01"/>
+          <mesh filename="file://$(find Kobuki_sim)/meshes/kobuki_base.stl" scale="0.01 0.01 0.01"/>
           <!--mesh filename="package://install/package_name/share/package_name/meshes/kobuki_base.stl" scale="0.01 0.01 0.01"/-->
           <!--cylinder radius="0.015" length="0.0206"/-->
